File: Pi_Interface.sch (EAGLE design)
At the start: 35 parts, among them IC1 A0 / GP, IC2 A1 / GS, J3 RASPI-40HAT, Q3 BSS138W-7-F, Q4 BSS138W-7-F, Q5 BSS138W-7-F, SW1 SPST_TACT-PT645, SW2 SPST_TACT-PT645

Commit message: Wired up opto-isolators
Parts:
- added R15, R16, R17, R18, R19, R20, R21, R22: (no value), rcl:R-EU_R0603
Connections:
- new net +3V3: J3.+3V3, J3.+3V3@2
- new net GNDIO: J-IN.5, OP1A.CT, OP1B.CT, OP1C.CT, OP1D.CT
- new net N$10: J-OUT.2, OP2B.E
- new net N$11: J-OUT.3, OP2C.E
- new net N$12: J-OUT.4, OP2D.E
- new net N$13: OP2A.AN, R15.2
- new net N$14: OP2B.AN, R16.2
- new net N$15: OP2C.AN, R17.2
- new net N$16: OP2D.AN, R18.2
- new net N$17: OP1A.AN, R19.1
- new net N$18: OP1B.AN, R20.1
- new net N$19: OP1C.AN, R21.1
- new net N$20: OP1D.AN, R22.1
- new net N$21: J-IN.1, R19.2
- new net N$22: J-IN.2, R20.2
- new net N$23: J-IN.3, R21.2
- new net N$24: J-IN.4, R22.2
- new net N$9: J-OUT.1, OP2A.E
- new net SCL: IC1.SCL, IC2.SCL, J3.BCM3-SCL
- new net SDA: IC1.SDA, IC2.SDA, J3.BCM2-SDA
- net +24V: now also OP2A.C, OP2B.C, OP2C.C, OP2D.C
- net GND: now also OP2A.CT, OP2B.CT, OP2C.CT, OP2D.CT; no longer J-IN.5
Other:
- moved on the sheet: J-IN, J-OUT, OP1A, OP1B, OP1C, OP1D, OP2A, OP2B, OP2C, OP2D

Commit message: Added 1206 resistor networks to minimize component count on board
Parts:
- removed R1, R10, R2, R3, R4, R8, R9: 100R, rcl:R-EU_R0603
- removed R15, R16, R17, R18: (no value), rcl:R-EU_R0603
- added R31, R32: 10k, rcl:R-EU_R0603
- added R33, R34: 330R, rcl:R-EU_R0603
- added RN1, RN2, RN5: 330R, resistor-network:R-NET4-1206C
- added RN3: 330R, resistor-network:R-NET4-1206
- added RN4: 10K, resistor-network:R-NET4-1206
- D1, D2: value 5.1V -> 3V6; device diode:ZENER-DIODESMB -> zener-diodes:ZENERSOD-123
- R11, R13: value 100R -> 10k
- R12, R14: value 100R -> 4k99
- R5, R6, R7: device rcl:R-EU_R0805 -> rcl:R-EU_R0603
Connections:
- new net IN1: J3.BCM5-GPCLK1, RN3D.1
- new net IN2: J3.BCM6-GPCLK2, RN3C.1
- new net IN3: J3.BCM7-CE1, RN3B.1
- new net IN4: J3.BCM8-CE0, RN3A.1
- new net N$25: OP1A.C, RN3D.2, RN4D.2
- new net N$26: R32.1, R34.2, SW2.S
- new net N$27: OP1B.C, RN3C.2, RN4C.2
- new net N$29: OP1C.C, RN3B.2, RN4B.2
- new net N$31: OP1D.C, RN3A.2, RN4A.2
- new net N$32: R31.1, R33.2, SW1.S
- new net OUT1: J3.BCM16, RN2D.1
- new net OUT2: J3.BCM17, RN2C.1
- new net OUT3: J3.BCM18-PCMCLK, RN2B.1
- new net OUT4: J3.BCM19-PCMFS, RN2A.1
- new net SERVO1: J3.BCM20-PCMDIN, RN1D.1
- new net SERVO2: J3.BCM21-PCMDOUT, RN1C.1
- new net SERVO3: J3.BCM22-SDIO-CLK, RN1B.1
- new net SERVO4: J3.BCM23-SDIO-CMD, RN1A.1
- new net SWITCH1: J3.BCM12-PWM0, R33.1
- new net SWITCH2: J3.BCM13-PWM1, R34.1
- net +3V3: now also IC1.VDD, IC2.VDD, R31.2, R32.2, RN4A.1, RN4B.1, RN4C.1, RN4D.1
- net +5V: no longer IC1.VDD, IC2.VDD
- net GND: now also OP1A.E, OP1B.E, OP1C.E, OP1D.E, SW1.P, SW2.P
- net N$1: now also RN1D.2; no longer R1.2
- net N$10: now also OP2C.E; no longer OP2B.E
- net N$11: now also OP2B.E; no longer OP2C.E
- net N$12: now also OP2A.E; no longer OP2D.E
- net N$13: now also OP2D.AN, RN2D.2; no longer OP2A.AN, R15.2
- net N$14: now also OP2C.AN, RN2C.2; no longer OP2B.AN, R16.2
- net N$15: now also OP2B.AN, RN2B.2; no longer OP2C.AN, R17.2
- net N$16: now also OP2A.AN, RN2A.2; no longer OP2D.AN, R18.2
- net N$2: now also RN1C.2; no longer R2.2
- net N$3: now also RN1B.2; no longer R3.2
- net N$4: now also RN1A.2; no longer R4.2
- net N$9: now also OP2D.E; no longer OP2A.E
- net RGB-B: now also J3.BCM11-SCK, RN5A.1; no longer R10.1
- net RGB-B-GATE: now also RN5A.2; no longer R10.2
- net RGB-G: now also J3.BCM10-MOSI, RN5C.1; no longer R9.1
- net RGB-G-GATE: now also RN5C.2; no longer R9.2
- net RGB-R: now also J3.BCM9-MISO, RN5B.1; no longer R8.1
- net RGB-R-GATE: now also RN5B.2; no longer R8.2
Other:
- moved on the sheet: D1, D2, IC1, IC2, J-AIN, J-IN, J-OUT, J-SRV1, J-SRV2, J-SRV3, J-SRV4, J-VSERVO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

Commit message: Changed Layout, added EEPROM
Parts:
- removed R19, R20, R21, R22: (no value), rcl:R-EU_R0603
- added C1: 100n, rcl:C-EUC0603
- added IC3: 24C32I-GW, eeprom:24C32I-GW
- added R1, R2: 3k9, rcl:R-EU_R0603
- added RN6: 560R, resistor-network:R-NET4-1206
- added WP: 0R, rcl:R-EU_R0603
Connections:
- net N$7 renamed AIN1
- net N$8 renamed AIN2
- new net ID_SCL: IC3.SCL, J3.BCM1-ID_SC, R1.1
- new net ID_SDA: IC3.SDA, J3.BCM0-ID_SD, R2.1
- new net WP: IC3.WP, WP.1
- net +3V3: now also C1.1, IC3.VCC, R1.2, R2.2, WP.2
- net GND: now also C1.2, IC3.A0, IC3.A1, IC3.A2, IC3.VSS
- net IN1: now also J3.BCM4-GPCLK0, RN3A.1, RN4A.2; no longer J3.BCM5-GPCLK1, RN3D.1
- net IN2: now also J3.BCM5-GPCLK1, RN3B.1, RN4B.2; no longer J3.BCM6-GPCLK2, RN3C.1
- net IN3: now also RN3C.1, RN4C.2; no longer RN3B.1
- net IN4: now also RN3D.1, RN4D.2; no longer RN3A.1
- net N$10: now also OP2B.E; no longer OP2C.E
- net N$11: now also OP2C.E; no longer OP2B.E
- net N$12: now also OP2D.E; no longer OP2A.E
- net N$17: now also RN6D.1; no longer R19.1
- net N$18: now also RN6C.1; no longer R20.1
- net N$19: now also RN6B.1; no longer R21.1
- net N$20: now also RN6A.1; no longer R22.1
- net N$21: now also RN6D.2; no longer R19.2
- net N$22: now also RN6C.2; no longer R20.2
- net N$23: now also RN6B.2; no longer R21.2
- net N$24: now also RN6A.2; no longer R22.2
- net N$25: now also OP1D.C; no longer OP1A.C, RN4D.2
- net N$27: now also OP1C.C; no longer OP1B.C, RN4C.2
- net N$29: now also OP1B.C; no longer OP1C.C, RN4B.2
- net N$31: now also OP1A.C; no longer OP1D.C, RN4A.2
- net N$9: now also OP2A.E; no longer OP2D.E
- net OUT1: now also J3.BCM18-PCMCLK, RN2A.1; no longer J3.BCM16, RN2D.1
- net OUT2: now also J3.BCM19-PCMFS, RN2B.1; no longer J3.BCM17, RN2C.1
- net OUT3: now also J3.BCM20-PCMDIN, RN2C.1; no longer J3.BCM18-PCMCLK, RN2B.1
- net OUT4: now also J3.BCM21-PCMDOUT, RN2D.1; no longer J3.BCM19-PCMFS, RN2A.1
- net SERVO1: now also J3.BCM22-SDIO-CLK; no longer J3.BCM20-PCMDIN
- net SERVO2: now also J3.BCM23-SDIO-CMD; no longer J3.BCM21-PCMDOUT
- net SERVO3: now also J3.BCM24-SDIO-DAT0; no longer J3.BCM22-SDIO-CLK
- net SERVO4: now also J3.BCM25-SDIO-DAT1; no longer J3.BCM23-SDIO-CMD
Other:
- moved on the sheet: OP2A, OP2B, OP2C, OP2D, RN2A, RN2B, RN2C, RN2D, RN3A, RN3B, RN3C, RN3D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
